File: hardware/f1oc/f1oc.kicad_pcb (KiCad board)
At the start: 2 copper layers, 33 x 33 mm, 54 parts, among them J1 Conn_01x04_Shielded, J3 Conn_01x04_Shielded, U1 STM32F103C8Tx, U2 DRV8316CRRGFR, U3 SN65HVD230, U4 MT6701CT, Y1 Crystal_GND24

Commit message: JLC pcb prototyping
Parts:
- added RN1: R_Pack04, Resistor_SMD:R_Array_Convex_4x0603, F.Cu at (122.3, 80.7)
- C5: value C_Polarized -> 10uF
- Y1: value Crystal_GND24 -> 8MHz
- moved C17 1.24 mm to (126.1, 81.1)
Connections:
- U2 pad 33: /MISO -> Net-(RN1-R4.1)
- U2 pad 34: /MOSI -> Net-(RN1-R3.1)
- U2 pad 35: /SCK -> Net-(RN1-R2.1)
- U2 pad 36: /CS_DRV -> Net-(RN1-R1.1)
Routing:
- net /CS_DRV: track 12.1 -> 5.79 mm
- net /SCK: track 19.9 -> 13.9 mm
- net Net-(RN1-R1.1): track 0.00 -> 5.76 mm
- net /MOSI: track 17.4 -> 11.8 mm
- net /MISO: track 17.6 -> 12.3 mm
- net Net-(RN1-R2.1): track 0.00 -> 4.22 mm
- net Net-(RN1-R3.1): track 0.00 -> 3.39 mm
- net Net-(RN1-R4.1): track 0.00 -> 2.70 mm
- net Net-(U2-VREF/ILIM): track 3.76 -> 2.20 mm
- net GND: vias 57 -> 61
