File: hardware/f1oc/f1oc.kicad_sch (KiCad schematic)
At the start: 54 parts, among them J1 Conn_01x04_Shielded, J3 Conn_01x04_Shielded, U1 STM32F103C8Tx, U2 DRV8316CRRGFR, U3 SN65HVD230, U4 MT6701CT, Y1 Crystal_GND24

Commit message: JLC pcb prototyping
Parts:
- added RN1: R_Pack04, Resistor_SMD:R_Array_Convex_4x0603, symbol Device:R_Pack04
- C5: value C_Polarized -> 10uF
- Y1: value Crystal_GND24 -> 8MHz
Connections:
- net CS_DRV: now also RN1.8 (R1.2); no longer U2.36 (NSCS)
- net MISO: now also RN1.5 (R4.2); no longer U2.33 (SDO)
- net MOSI: now also RN1.6 (R3.2); no longer U2.34 (SDI)
- net SCK: now also RN1.7 (R2.2); no longer U2.35 (SCLK)
- new net: RN1.4 (R4.1), U2.33 (SDO)
- new net: RN1.3 (R3.1), U2.34 (SDI)
- new net: RN1.2 (R2.1), U2.35 (SCLK)
- new net: RN1.1 (R1.1), U2.36 (NSCS)
Other:
- moved on the sheet: C14, C15, C16, C17, R4, R5, R6
